File: Pac-Man/Pac-Man.kicad_sch (KiCad schematic)
At the start: 9 parts, among them U22 Controls, U33 74154, U34 74154, U37 74LS32, U39 Start, U40 HDSP-7401

Commit message: Add files via upload
Connections:
- net at U32. (RD9): now also U33.9 (~{S8})
Changed lines of the file:
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@@
 	)
 	(symbol
-		(lib_name "Pasquale:debounced_buttons")
 		(lib_id "Pasquale:debounced_buttons")
 		(at 45.72 58.42 90)
@@
 	)
 	(symbol
-		(lib_name "Pasquale:debounced_buttons")
 		(lib_id "Pasquale:debounced_buttons")
 		(at 64.77 29.21 0)
