File: Pac-Man/Pac_Man_Movement.kicad_sch (KiCad schematic)
At the start: 21 parts, among them U1 74LS32, U10 74LS04, U11 74LS04, U12 74LS04, U13 74LS04, U14 74LS04, U15 74LS04, U16 74LS194, U17 74LS04, U18 74LS04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

Commit message: Add files via upload
Parts:
- removed unit 1 of U13
- removed U14, U6: 74LS04, symbol 74xx:74LS04
- removed unit 1 of U5
Connections:
- net at U21.7 (A3), U4.12 (Q3), U9.3: no longer U11.3, U21.10 (A0), U4.15 (Q0)
- net at U7.3: now also U5.4
- net at U8.3: now also U13.3
- net at U13.4: now also U15.3
- net at U5.3: now also U3.3
- new net: U11.3, U21.10 (A0), U4.15 (Q0)
